Commit message: added changes from Cleanup #5

File: thmho_heatmap_generator/urdf/lab.xacro (robot description, xacro)
@@ -1,5 +1,5 @@
 <?xml version="1.0"?>
 <robot xmlns:xacro="http://www.ros.org/wiki/xacro" name="lab_model">
-  <xacro:include filename="$(find thmho_heatmap_generator)/urdf/laser.plugins.xacro" />
+  <xacro:include filename="$(find factory_sim)/urdf/laser.plugins.xacro" />
   <xacro:property name="laser_size_x" value="0.03"/>
   <xacro:property name="laser_size_y" value="0.03"/>
@@ -82,5 +82,5 @@
     <visual>
       <geometry>
-        <mesh filename="package://thmho_heatmap_generator/meshes/hokuyo.dae"/>
+        <mesh filename="package://factory_sim/meshes/hokuyo.dae"/>
         <!--box size="${laser_size_x} ${laser_size_y} ${laser_size_z}"/-->
       </geometry>
@@ -98,5 +98,5 @@
     <visual>
       <geometry>
-        <mesh filename="package://thmho_heatmap_generator/meshes/hokuyo.dae"/>
+        <mesh filename="package://factory_sim/meshes/hokuyo.dae"/>
         <!--box size="${laser_size_x} ${laser_size_y} ${laser_size_z}"/-->
       </geometry>
